File: minimal_ad74413r/minimal_ad74413r.kicad_sch (KiCad schematic)
At the start: 60 parts, among them J1 FW-02-03-G-D-085-315, J2 FW-02-03-G-D-085-315, J3 FW-02-03-G-D-085-155, J4 FW-02-03-G-D-085-155, J5 FW-02-03-G-D-085-315, J6 FW-02-03-G-D-085-315, J7 FW-14-03-G-D-085-155, U1 AD74413RBCPZ

Commit message: Backup
Parts:
- J1, J2, J5, J6: value FW-02-03-G-D-085-315 -> FW-02-03-G-D-085-155; footprint connector_footprints:FW-02-03-G-D-085-315 -> connector_footprints:FW-02-03-G-D-085-155; symbol UNITED_CONNECTORS_DATA_BASE:J_FW-02-03-G-D-085-315 -> UNITED_CONNECTORS_DATA_BASE:J_FW-02-03-G-D-085-155; MPN FW-02-03-G-D-085-315 -> FW-02-03-G-D-085-155; Series FW-xx-03-G-D-085-315 -> FW-xx-03-G-D-085-155; Symbol Name J_FW-02-03-G-D-085-315 -> J_FW-02-03-G-D-085-155; Trustedparts Search https://www.trustedparts.com/en/search/FW-02-03-G-D-085-315 -> https://www.trustedparts.com/en/search/FW-02-03-G-D-085-155
Changed lines of the file:
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@@
 	)
 	(symbol
-		(lib_id "UNITED_CONNECTORS_DATA_BASE:J_FW-02-03-G-D-085-315")
+		(lib_id "UNITED_CONNECTORS_DATA_BASE:J_FW-02-03-G-D-085-155")
 		(at 285.75 207.01 90)
 		(mirror x)
@@
 			)
 		)
-		(property "Value" "FW-02-03-G-D-085-315"
+		(property "Value" "FW-02-03-G-D-085-155"
 			(at 290.83 208.2799 90)
 			(effects
@@
 			)
 		)
-		(property "Footprint" "connector_footprints:FW-02-03-G-D-085-315"
+		(property "Footprint" "connector_footprints:FW-02-03-G-D-085-155"
 			(at 293.37 212.09 0)
 			(show_name yes)
@@
 			)
 		)
-		(property "Description" "Samtec FW-xx-03-G-D-085-315 series,  2 positions connector,  1.27 mm pitch,  Black,  Vertical mounting,  5.2 A,  300 V,  Surface Mount,  Gold plated"
+		(property "Description" "Samtec FW-xx-03-G-D-085-155 series,  2 positions connector,  1.27 mm pitch,  Black,  Vertical mounting,  5.2 A,  300 V,  Surface Mount,  Gold plated"
 			(at 298.45 212.09 0)
 			(show_name yes)
@@
 			)
 		)
-		(property "MPN" "FW-02-03-G-D-085-315"
+		(property "MPN" "FW-02-03-G-D-085-155"
 			(at 308.61 212.09 0)
 			(show_name yes)
@@
 			)
 		)
-		(property "Series" "FW-xx-03-G-D-085-315"
+		(property "Series" "FW-xx-03-G-D-085-155"
 			(at 326.39 212.09 0)
 			(show_name yes)
@@
 			)
 		)
-		(property "Symbol Name" "J_FW-02-03-G-D-085-315"
+		(property "Symbol Name" "J_FW-02-03-G-D-085-155"
 			(at 328.93 212.09 0)
 			(show_name yes)
@@
 			)
 		)
-		(property "Trustedparts Search" "https://www.trustedparts.com/en/search/FW-02-03-G-D-085-315"
+		(property "Trustedparts Search" "https://www.trustedparts.com/en/search/FW-02-03-G-D-085-155"
 			(at 331.47 212.09 0)
 			(show_name yes)
@@
 	)
 	(symbol
-		(lib_id "UNITED_CONNECTORS_DATA_BASE:J_FW-02-03-G-D-085-315")
+		(lib_id "UNITED_CONNECTORS_DATA_BASE:J_FW-02-03-G-D-085-155")
 		(at 285.75 151.13 90)
 		(mirror x)
@@
 			)
 		)
-		(property "Value" "FW-02-03-G-D-085-315"
+		(property "Value" "FW-02-03-G-D-085-155"
 			(at 290.83 152.3999 90)
 			(effects
@@
 			)
 		)
-		(property "Footprint" "connector_footprints:FW-02-03-G-D-085-315"
+		(property "Footprint" "connector_footprints:FW-02-03-G-D-085-155"
 			(at 293.37 156.21 0)
 			(show_name yes)
@@
 			)
 		)
-		(property "Description" "Samtec FW-xx-03-G-D-085-315 series,  2 positions connector,  1.27 mm pitch,  Black,  Vertical mounting,  5.2 A,  300 V,  Surface Mount,  Gold plated"
+		(property "Description" "Samtec FW-xx-03-G-D-085-155 series,  2 positions connector,  1.27 mm pitch,  Black,  Vertical mounting,  5.2 A,  300 V,  Surface Mount,  Gold plated"
 			(at 298.45 156.21 0)
 			(show_name yes)
@@
 			)
 		)
-		(property "MPN" "FW-02-03-G-D-085-315"
+		(property "MPN" "FW-02-03-G-D-085-155"
 			(at 308.61 156.21 0)
 			(show_name yes)
@@
 			)
 		)
-		(property "Series" "FW-xx-03-G-D-085-315"
+		(property "Series" "FW-xx-03-G-D-085-155"
 			(at 326.39 156.21 0)
 			(show_name yes)
@@
 			)
 		)
-		(property "Symbol Name" "J_FW-02-03-G-D-085-315"
+		(property "Symbol Name" "J_FW-02-03-G-D-085-155"
 			(at 328.93 156.21 0)
 			(show_name yes)
@@
 			)
 		)
-		(property "Trustedparts Search" "https://www.trustedparts.com/en/search/FW-02-03-G-D-085-315"
+		(property "Trustedparts Search" "https://www.trustedparts.com/en/search/FW-02-03-G-D-085-155"
 			(at 331.47 156.21 0)
 			(show_name yes)
@@
 	)
 	(symbol
-		(lib_id "UNITED_CONNECTORS_DATA_BASE:J_FW-02-03-G-D-085-315")
+		(lib_id "UNITED_CONNECTORS_DATA_BASE:J_FW-02-03-G-D-085-155")
 		(at 285.75 179.07 270)
 		(mirror x)
@@
 			)
 		)
-		(property "Value" "FW-02-03-G-D-085-315"
+		(property "Value" "FW-02-03-G-D-085-155"
 			(at 290.83 180.3399 90)
 			(effects
@@
 			)
 		)
-		(property "Footprint" "connector_footprints:FW-02-03-G-D-085-315"
+		(property "Footprint" "connector_footprints:FW-02-03-G-D-085-155"
 			(at 278.13 173.99 0)
 			(show_name yes)
@@
 			)
 		)
-		(property "Description" "Samtec FW-xx-03-G-D-085-315 series,  2 positions connector,  1.27 mm pitch,  Black,  Vertical mounting,  5.2 A,  300 V,  Surface Mount,  Gold plated"
+		(property "Description" "Samtec FW-xx-03-G-D-085-155 series,  2 positions connector,  1.27 mm pitch,  Black,  Vertical mounting,  5.2 A,  300 V,  Surface Mount,  Gold plated"
 			(at 273.05 173.99 0)
 			(show_name yes)
@@
 			)
 		)
-		(property "MPN" "FW-02-03-G-D-085-315"
+		(property "MPN" "FW-02-03-G-D-085-155"
 			(at 262.89 173.99 0)
 			(show_name yes)
@@
 			)
 		)
-		(property "Series" "FW-xx-03-G-D-085-315"
+		(property "Series" "FW-xx-03-G-D-085-155"
 			(at 245.11 173.99 0)
 			(show_name yes)
@@
 			)
 		)
-		(property "Symbol Name" "J_FW-02-03-G-D-085-315"
+		(property "Symbol Name" "J_FW-02-03-G-D-085-155"
 			(at 242.57 173.99 0)
 			(show_name yes)
@@
 			)
 		)
-		(property "Trustedparts Search" "https://www.trustedparts.com/en/search/FW-02-03-G-D-085-315"
+		(property "Trustedparts Search" "https://www.trustedparts.com/en/search/FW-02-03-G-D-085-155"
 			(at 240.03 173.99 0)
 			(show_name yes)
@@
 	)
 	(symbol
-		(lib_id "UNITED_CONNECTORS_DATA_BASE:J_FW-02-03-G-D-085-315")
+		(lib_id "UNITED_CONNECTORS_DATA_BASE:J_FW-02-03-G-D-085-155")
 		(at 285.75 123.19 270)
 		(mirror x)
@@
 			)
 		)
-		(property "Value" "FW-02-03-G-D-085-315"
+		(property "Value" "FW-02-03-G-D-085-155"
 			(at 290.83 124.4599 90)
 			(effects
@@
 			)
 		)
-		(property "Footprint" "connector_footprints:FW-02-03-G-D-085-315"
+		(property "Footprint" "connector_footprints:FW-02-03-G-D-085-155"
 			(at 278.13 118.11 0)
 			(show_name yes)
@@
 			)
 		)
-		(property "Description" "Samtec FW-xx-03-G-D-085-315 series,  2 positions connector,  1.27 mm pitch,  Black,  Vertical mounting,  5.2 A,  300 V,  Surface Mount,  Gold plated"
+		(property "Description" "Samtec FW-xx-03-G-D-085-155 series,  2 positions connector,  1.27 mm pitch,  Black,  Vertical mounting,  5.2 A,  300 V,  Surface Mount,  Gold plated"
 			(at 273.05 118.11 0)
 			(show_name yes)
@@
 			)
 		)
-		(property "MPN" "FW-02-03-G-D-085-315"
+		(property "MPN" "FW-02-03-G-D-085-155"
 			(at 262.89 118.11 0)
 			(show_name yes)
@@
 			)
 		)
-		(property "Series" "FW-xx-03-G-D-085-315"
+		(property "Series" "FW-xx-03-G-D-085-155"
 			(at 245.11 118.11 0)
 			(show_name yes)
@@
 			)
 		)
-		(property "Symbol Name" "J_FW-02-03-G-D-085-315"
+		(property "Symbol Name" "J_FW-02-03-G-D-085-155"
 			(at 242.57 118.11 0)
 			(show_name yes)
@@
 			)
 		)
-		(property "Trustedparts Search" "https://www.trustedparts.com/en/search/FW-02-03-G-D-085-315"
+		(property "Trustedparts Search" "https://www.trustedparts.com/en/search/FW-02-03-G-D-085-155"
 			(at 240.03 118.11 0)
 			(show_name yes)
@@
 		(fields_autoplaced yes)
 		(property "Reference" "J4"
-			(at 161.29 30.4799 90)
+			(at 171.45 30.4799 90)
 			(effects
 				(font
 					(size 1.27 1.27)
 				)
-				(justify right)
+				(justify left)
 			)
 		)
 		(property "Value" "FW-02-03-G-D-085-155"
-			(at 161.29 33.0199 90)
+			(at 171.45 33.0199 90)
 			(effects
 				(font
 					(size 1.27 1.27)
 				)
-				(justify right)
+				(justify left)
 			)
 		)

Commit message: Update subproject commit for KiCAD_Symbol_Generator
Parts:
- C1, C17, C18, C2: value 10 uF -> 10 µF; 3dviewer Link (none) -> https://3dviewer.net/index.html#model=https://github.com/io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; Capacitor Type (none) -> Ceramic
- C14, C16, C19, C20, C29, C3, C30, C31, C5: value 0.1uF -> 100 nF; 3dviewer Link (none) -> https://3dviewer.net/index.html#model=https://github.com/io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; Capacitor Type (none) -> Ceramic
- C15, C32: value 2.2 uF -> 2.2 µF; 3dviewer Link (none) -> https://3dviewer.net/index.html#model=https://github.com/io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; Capacitor Type (none) -> Ceramic
- C4: value 0.33 uF -> 330 nF; 3dviewer Link (none) -> https://3dviewer.net/index.html#model=https://github.com/io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; Capacitor Type (none) -> Ceramic

Commit message: Switch to KiCad 9
Changed lines of the file:
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@@
 (kicad_sch
-	(version 20231120)
+	(version 20250114)
 	(generator "eeschema")
-	(generator_version "8.0")
+	(generator_version "9.0")
 	(paper "A3")
 	(junction
@@
 		(at 241.3 170.18)
 		(size 27.94 22.86)
+		(exclude_from_sim no)
+		(in_bom yes)
+		(on_board yes)
+		(dnp no)
 		(fields_autoplaced yes)
 		(stroke
@@
 		(at 241.3 114.3)
 		(size 27.94 22.86)
+		(exclude_from_sim no)
+		(in_bom yes)
+		(on_board yes)
+		(dnp no)
 		(fields_autoplaced yes)
 		(stroke
@@
 		(at 241.3 198.12)
 		(size 27.94 22.86)
+		(exclude_from_sim no)
+		(in_bom yes)
+		(on_board yes)
+		(dnp no)
 		(fields_autoplaced yes)
 		(stroke
@@
 		(at 241.3 142.24)
 		(size 27.94 22.86)
+		(exclude_from_sim no)
+		(in_bom yes)
+		(on_board yes)
+		(dnp no)
 		(fields_autoplaced yes)
 		(stroke
@@
 		)
 	)
+	(embedded_fonts no)
 )
