File: minimal_ad74413r/Front End Channel 1.kicad_sch (KiCad schematic)
At the start: 11 parts, among them Q3 ZXMP6A17E6TA

Commit message: Minor updates
Parts:
- renumbered C11 to C10, C9 to C12, C10 to C6, C12 to C8, CR3 to CR1, Q3 to Q2, R11 to R1, R12 to R3, R15 to R5, R13 to R7, R14 to R9
Changed lines of the file:
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@@
 		(dnp no)
 		(fields_autoplaced yes)
-		(property "Reference" "Q3"
+		(property "Reference" "Q2"
 			(at 201.93 187.9599 90)
 			(effects
@@
 			(project "minimal_ad74413r"
 				(path "/3d1a8eae-9f4e-4ae3-8a80-a6e3408e9f8d/215a75b8-84cc-467b-b211-24faa4125349"
+					(reference "Q2")
+					(unit 1)
+				)
+				(path "/3d1a8eae-9f4e-4ae3-8a80-a6e3408e9f8d/471bb7b7-cd79-4b45-b5fa-ce18ba37980a"
 					(reference "Q3")
-					(unit 1)
-				)
-				(path "/3d1a8eae-9f4e-4ae3-8a80-a6e3408e9f8d/471bb7b7-cd79-4b45-b5fa-ce18ba37980a"
-					(reference "Q1")
 					(unit 1)
 				)
@@
 				)
 				(path "/3d1a8eae-9f4e-4ae3-8a80-a6e3408e9f8d/ed3c01a7-dc5a-420d-9436-94dfdef482d0"
-					(reference "Q2")
+					(reference "Q1")
 					(unit 1)
 				)
@@
 		(dnp no)
 		(fields_autoplaced yes)
-		(property "Reference" "C9"
+		(property "Reference" "C12"
 			(at 189.23 132.0799 90)
 			(effects
@@
 			(project "minimal_ad74413r"
 				(path "/3d1a8eae-9f4e-4ae3-8a80-a6e3408e9f8d/215a75b8-84cc-467b-b211-24faa4125349"
-					(reference "C9")
+					(reference "C12")
 					(unit 1)
 				)
 				(path "/3d1a8eae-9f4e-4ae3-8a80-a6e3408e9f8d/471bb7b7-cd79-4b45-b5fa-ce18ba37980a"
-					(reference "C1")
+					(reference "C22")
 					(unit 1)
 				)
 				(path "/3d1a8eae-9f4e-4ae3-8a80-a6e3408e9f8d/77ed2068-19f4-4838-81a2-88ec2b717aa2"
+					(reference "C21")
+					(unit 1)
+				)
+				(path "/3d1a8eae-9f4e-4ae3-8a80-a6e3408e9f8d/ed3c01a7-dc5a-420d-9436-94dfdef482d0"
 					(reference "C13")
-					(unit 1)
-				)
-				(path "/3d1a8eae-9f4e-4ae3-8a80-a6e3408e9f8d/ed3c01a7-dc5a-420d-9436-94dfdef482d0"
-					(reference "C5")
 					(unit 1)
 				)
@@
 		(dnp no)
 		(fields_autoplaced yes)
-		(property "Reference" "R11"
+		(property "Reference" "R1"
 			(at 198.12 146.05 0)
 			(effects
@@
 			(project "minimal_ad74413r"
 				(path "/3d1a8eae-9f4e-4ae3-8a80-a6e3408e9f8d/215a75b8-84cc-467b-b211-24faa4125349"
-					(reference "R11")
+					(reference "R1")
 					(unit 1)
 				)
 				(path "/3d1a8eae-9f4e-4ae3-8a80-a6e3408e9f8d/471bb7b7-cd79-4b45-b5fa-ce18ba37980a"
-					(reference "R1")
+					(reference "R20")
 					(unit 1)
 				)
 				(path "/3d1a8eae-9f4e-4ae3-8a80-a6e3408e9f8d/77ed2068-19f4-4838-81a2-88ec2b717aa2"
-					(reference "R16")
+					(reference "R19")
 					(unit 1)
 				)
 				(path "/3d1a8eae-9f4e-4ae3-8a80-a6e3408e9f8d/ed3c01a7-dc5a-420d-9436-94dfdef482d0"
-					(reference "R6")
+					(reference "R2")
 					(unit 1)
 				)
@@
 		(dnp no)
 		(fields_autoplaced yes)
-		(property "Reference" "C11"
+		(property "Reference" "C10"
 			(at 199.39 93.98 0)
 			(effects
@@
 			(project "minimal_ad74413r"
 				(path "/3d1a8eae-9f4e-4ae3-8a80-a6e3408e9f8d/215a75b8-84cc-467b-b211-24faa4125349"
+					(reference "C10")
+					(unit 1)
+				)
+				(path "/3d1a8eae-9f4e-4ae3-8a80-a6e3408e9f8d/471bb7b7-cd79-4b45-b5fa-ce18ba37980a"
+					(reference "C24")
+					(unit 1)
+				)
+				(path "/3d1a8eae-9f4e-4ae3-8a80-a6e3408e9f8d/77ed2068-19f4-4838-81a2-88ec2b717aa2"
+					(reference "C23")
+					(unit 1)
+				)
+				(path "/3d1a8eae-9f4e-4ae3-8a80-a6e3408e9f8d/ed3c01a7-dc5a-420d-9436-94dfdef482d0"
 					(reference "C11")
-					(unit 1)
-				)
-				(path "/3d1a8eae-9f4e-4ae3-8a80-a6e3408e9f8d/471bb7b7-cd79-4b45-b5fa-ce18ba37980a"
-					(reference "C3")
-					(unit 1)
-				)
-				(path "/3d1a8eae-9f4e-4ae3-8a80-a6e3408e9f8d/77ed2068-19f4-4838-81a2-88ec2b717aa2"
-					(reference "C15")
-					(unit 1)
-				)
-				(path "/3d1a8eae-9f4e-4ae3-8a80-a6e3408e9f8d/ed3c01a7-dc5a-420d-9436-94dfdef482d0"
-					(reference "C7")
 					(unit 1)
 				)
@@
 		(dnp no)
 		(fields_autoplaced yes)
-		(property "Reference" "R15"
+		(property "Reference" "R5"
 			(at 218.44 138.4299 90)
 			(effects
@@
 			(project "minimal_ad74413r"
 				(path "/3d1a8eae-9f4e-4ae3-8a80-a6e3408e9f8d/215a75b8-84cc-467b-b211-24faa4125349"
+					(reference "R5")
+					(unit 1)
+				)
+				(path "/3d1a8eae-9f4e-4ae3-8a80-a6e3408e9f8d/471bb7b7-cd79-4b45-b5fa-ce18ba37980a"
+					(reference "R16")
+					(unit 1)
+				)
+				(path "/3d1a8eae-9f4e-4ae3-8a80-a6e3408e9f8d/77ed2068-19f4-4838-81a2-88ec2b717aa2"
 					(reference "R15")
 					(unit 1)
 				)
-				(path "/3d1a8eae-9f4e-4ae3-8a80-a6e3408e9f8d/471bb7b7-cd79-4b45-b5fa-ce18ba37980a"
-					(reference "R5")
-					(unit 1)
-				)
-				(path "/3d1a8eae-9f4e-4ae3-8a80-a6e3408e9f8d/77ed2068-19f4-4838-81a2-88ec2b717aa2"
-					(reference "R20")
-					(unit 1)
-				)
 				(path "/3d1a8eae-9f4e-4ae3-8a80-a6e3408e9f8d/ed3c01a7-dc5a-420d-9436-94dfdef482d0"
-					(reference "R10")
+					(reference "R6")
 					(unit 1)
 				)
@@
 		(dnp no)
 		(fields_autoplaced yes)
-		(property "Reference" "C12"
+		(property "Reference" "C8"
 			(at 232.41 113.0299 90)
 			(effects
@@
 			(project "minimal_ad74413r"
 				(path "/3d1a8eae-9f4e-4ae3-8a80-a6e3408e9f8d/215a75b8-84cc-467b-b211-24faa4125349"
-					(reference "C12")
+					(reference "C8")
 					(unit 1)
 				)
 				(path "/3d1a8eae-9f4e-4ae3-8a80-a6e3408e9f8d/471bb7b7-cd79-4b45-b5fa-ce18ba37980a"
-					(reference "C4")
+					(reference "C26")
 					(unit 1)
 				)
 				(path "/3d1a8eae-9f4e-4ae3-8a80-a6e3408e9f8d/77ed2068-19f4-4838-81a2-88ec2b717aa2"
-					(reference "C16")
+					(reference "C25")
 					(unit 1)
 				)
 				(path "/3d1a8eae-9f4e-4ae3-8a80-a6e3408e9f8d/ed3c01a7-dc5a-420d-9436-94dfdef482d0"
-					(reference "C8")
+					(reference "C9")
 					(unit 1)
 				)
@@
 		(dnp no)
 		(fields_autoplaced yes)
-		(property "Reference" "C10"
+		(property "Reference" "C6"
 			(at 189.23 170.1799 90)
 			(effects
@@
 			(project "minimal_ad74413r"
 				(path "/3d1a8eae-9f4e-4ae3-8a80-a6e3408e9f8d/215a75b8-84cc-467b-b211-24faa4125349"
-					(reference "C10")
+					(reference "C6")
 					(unit 1)
 				)
 				(path "/3d1a8eae-9f4e-4ae3-8a80-a6e3408e9f8d/471bb7b7-cd79-4b45-b5fa-ce18ba37980a"
-					(reference "C2")
+					(reference "C28")
 					(unit 1)
 				)
 				(path "/3d1a8eae-9f4e-4ae3-8a80-a6e3408e9f8d/77ed2068-19f4-4838-81a2-88ec2b717aa2"
-					(reference "C14")
+					(reference "C27")
 					(unit 1)
 				)
 				(path "/3d1a8eae-9f4e-4ae3-8a80-a6e3408e9f8d/ed3c01a7-dc5a-420d-9436-94dfdef482d0"
-					(reference "C6")
+					(reference "C7")
 					(unit 1)
 				)
@@
 		(dnp no)
 		(fields_autoplaced yes)
-		(property "Reference" "R12"
+		(property "Reference" "R3"
 			(at 198.12 158.75 0)
 			(effects
@@
 			(project "minimal_ad74413r"
 				(path "/3d1a8eae-9f4e-4ae3-8a80-a6e3408e9f8d/215a75b8-84cc-467b-b211-24faa4125349"
-					(reference "R12")
+					(reference "R3")
 					(unit 1)
 				)
 				(path "/3d1a8eae-9f4e-4ae3-8a80-a6e3408e9f8d/471bb7b7-cd79-4b45-b5fa-ce18ba37980a"
-					(reference "R2")
+					(reference "R18")
 					(unit 1)
 				)
@@
 				)
 				(path "/3d1a8eae-9f4e-4ae3-8a80-a6e3408e9f8d/ed3c01a7-dc5a-420d-9436-94dfdef482d0"
-					(reference "R7")
+					(reference "R4")
 					(unit 1)
 				)
@@
 		(dnp no)
 		(fields_autoplaced yes)
-		(property "Reference" "R13"
+		(property "Reference" "R7"
 			(at 199.39 107.95 0)
 			(effects
@@
 			(project "minimal_ad74413r"
 				(path "/3d1a8eae-9f4e-4ae3-8a80-a6e3408e9f8d/215a75b8-84cc-467b-b211-24faa4125349"
+					(reference "R7")
+					(unit 1)
+				)
+				(path "/3d1a8eae-9f4e-4ae3-8a80-a6e3408e9f8d/471bb7b7-cd79-4b45-b5fa-ce18ba37980a"
+					(reference "R14")
+					(unit 1)
+				)
+				(path "/3d1a8eae-9f4e-4ae3-8a80-a6e3408e9f8d/77ed2068-19f4-4838-81a2-88ec2b717aa2"
 					(reference "R13")
-					(unit 1)
-				)
-				(path "/3d1a8eae-9f4e-4ae3-8a80-a6e3408e9f8d/471bb7b7-cd79-4b45-b5fa-ce18ba37980a"
-					(reference "R3")
-					(unit 1)
-				)
-				(path "/3d1a8eae-9f4e-4ae3-8a80-a6e3408e9f8d/77ed2068-19f4-4838-81a2-88ec2b717aa2"
-					(reference "R18")
 					(unit 1)
 				)
@@
 		(on_board yes)
 		(dnp no)
-		(property "Reference" "CR3"
+		(property "Reference" "CR1"
 			(at 215.9 181.61 0)
 			(effects
@@
 			(project "minimal_ad74413r"
 				(path "/3d1a8eae-9f4e-4ae3-8a80-a6e3408e9f8d/215a75b8-84cc-467b-b211-24faa4125349"
+					(reference "CR1")
+					(unit 1)
+				)
+				(path "/3d1a8eae-9f4e-4ae3-8a80-a6e3408e9f8d/471bb7b7-cd79-4b45-b5fa-ce18ba37980a"
+					(reference "CR4")
+					(unit 1)
+				)
+				(path "/3d1a8eae-9f4e-4ae3-8a80-a6e3408e9f8d/77ed2068-19f4-4838-81a2-88ec2b717aa2"
 					(reference "CR3")
-					(unit 1)
-				)
-				(path "/3d1a8eae-9f4e-4ae3-8a80-a6e3408e9f8d/471bb7b7-cd79-4b45-b5fa-ce18ba37980a"
-					(reference "CR1")
-					(unit 1)
-				)
-				(path "/3d1a8eae-9f4e-4ae3-8a80-a6e3408e9f8d/77ed2068-19f4-4838-81a2-88ec2b717aa2"
-					(reference "CR4")
 					(unit 1)
 				)
@@
 		(dnp no)
 		(fields_autoplaced yes)
-		(property "Reference" "R14"
+		(property "Reference" "R9"
 			(at 199.39 120.65 0)
 			(effects
@@
 			(project "minimal_ad74413r"
 				(path "/3d1a8eae-9f4e-4ae3-8a80-a6e3408e9f8d/215a75b8-84cc-467b-b211-24faa4125349"
-					(reference "R14")
+					(reference "R9")
 					(unit 1)
 				)
 				(path "/3d1a8eae-9f4e-4ae3-8a80-a6e3408e9f8d/471bb7b7-cd79-4b45-b5fa-ce18ba37980a"
-					(reference "R4")
+					(reference "R12")
 					(unit 1)
 				)
 				(path "/3d1a8eae-9f4e-4ae3-8a80-a6e3408e9f8d/77ed2068-19f4-4838-81a2-88ec2b717aa2"
-					(reference "R19")
+					(reference "R11")
 					(unit 1)
 				)
 				(path "/3d1a8eae-9f4e-4ae3-8a80-a6e3408e9f8d/ed3c01a7-dc5a-420d-9436-94dfdef482d0"
-					(reference "R9")
-					(unit 1)
-				)
+					(reference "R10")
+					(unit 1)
+				)

Commit message: Update subproject commit for KiCAD_Symbol_Generator
Parts:
- C10: 3dviewer Link (none) -> https://3dviewer.net/index.html#model=https://github.com/io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; Capacitor Type (none) -> Ceramic
- C12, C6, C8: value 0.01 uF -> 10 nF; 3dviewer Link (none) -> https://3dviewer.net/index.html#model=https://github.com/io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; Capacitor Type (none) -> Ceramic
- CR1: value SBAV99WT1G -> 100 V; Manufacturer Kingbright -> Onsemi
- Q2: value ZXMP6A17E6TA -> -60 V; 3dviewer Link (none) -> https://3dviewer.net/index.html#model=https://github.com/io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
- R1, R7: value 2k -> 2 kΩ; 3dviewer Link (none) -> https://3dviewer.net/index.html#model=https://github.com/io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; Component Type (none) -> Resistor
- R3, R9: value 10k -> 10 kΩ; 3dviewer Link (none) -> https://3dviewer.net/index.html#model=https://github.com/io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; Component Type (none) -> Resistor
- R5: value 100 -> 100 Ω; 3dviewer Link (none) -> https://3dviewer.net/index.html#model=https://github.com/io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; Component Type (none) -> Resistor

Commit message: Switch to KiCad 9
Parts:
- renumbered C12 to C22, C10 to C24, C8 to C25, C6 to C28, CR1 to CR4, Q2 to Q3, R9 to R12, R7 to R14, R5 to R15, R3 to R18, R1 to R20
Changed lines of the file:
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@@
 (kicad_sch
-	(version 20231120)
+	(version 20250114)
 	(generator "eeschema")
-	(generator_version "8.0")
+	(generator_version "9.0")
 	(paper "A3")
 	(junction
@@
 		(dnp no)
 		(fields_autoplaced yes)
-		(property "Reference" "Q2"
+		(property "Reference" "Q3"
 			(at 201.93 187.9599 90)
 			(effects
@@
 		(dnp no)
 		(fields_autoplaced yes)
-		(property "Reference" "C12"
+		(property "Reference" "C22"
 			(at 189.23 132.0799 90)
 			(effects
@@
 		(dnp no)
 		(fields_autoplaced yes)
-		(property "Reference" "#PWR17"
+		(property "Reference" "#PWR11"
 			(at 185.42 182.88 0)
 			(effects
@@
 		(dnp no)
 		(fields_autoplaced yes)
-		(property "Reference" "R1"
+		(property "Reference" "R20"
 			(at 198.12 146.05 0)
 			(effects
@@
 		(dnp no)
 		(fields_autoplaced yes)
-		(property "Reference" "#PWR16"
+		(property "Reference" "#PWR10"
 			(at 185.42 144.78 0)
 			(effects
@@
 		(dnp no)
 		(fields_autoplaced yes)
-		(property "Reference" "C10"
+		(property "Reference" "C24"
 			(at 199.39 93.98 0)
 			(effects
@@
 		(dnp no)
 		(fields_autoplaced yes)
-		(property "Reference" "R5"
+		(property "Reference" "R15"
 			(at 218.44 138.4299 90)
 			(effects
@@
 		(dnp no)
 		(fields_autoplaced yes)
-		(property "Reference" "C8"
+		(property "Reference" "C25"
 			(at 232.41 113.0299 90)
 			(effects
@@
 		(dnp no)
 		(fields_autoplaced yes)
-		(property "Reference" "C6"
+		(property "Reference" "C28"
 			(at 189.23 170.1799 90)
 			(effects
@@
 		(dnp no)
 		(fields_autoplaced yes)
-		(property "Reference" "R3"
+		(property "Reference" "R18"
 			(at 198.12 158.75 0)
 			(effects
@@
 		(dnp no)
 		(fields_autoplaced yes)
-		(property "Reference" "R7"
+		(property "Reference" "R14"
 			(at 199.39 107.95 0)
 			(effects
@@
 		(dnp no)
 		(fields_autoplaced yes)
-		(property "Reference" "#PWR18"
+		(property "Reference" "#PWR13"
 			(at 228.6 132.08 0)
 			(effects
@@
 		(on_board yes)
 		(dnp no)
-		(property "Reference" "CR1"
+		(property "Reference" "CR4"
 			(at 215.9 181.61 0)
 			(effects
@@
 		(dnp no)
 		(fields_autoplaced yes)
-		(property "Reference" "R9"
+		(property "Reference" "R12"
 			(at 199.39 120.65 0)
 			(effects

Commit message: Development backup
Parts:
- added D12: 40 V, diode_footprints:DO-214AB-2, symbol UNITED_DIODES_DATA_BASE:D_SMCJ40A-CA
Connections:
- net AIO: now also D12.1
- net GNDA: now also D12.2

Commit message: Development backup
Parts:
- renumbered D12 to D4
Changed lines of the file:
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@@
 		(dnp no)
 		(fields_autoplaced yes)
-		(property "Reference" "#PWR11"
+		(property "Reference" "#PWR52"
 			(at 185.42 182.88 0)
 			(effects
@@
 			(project "minimal_ad74413r"
 				(path "/3d1a8eae-9f4e-4ae3-8a80-a6e3408e9f8d/215a75b8-84cc-467b-b211-24faa4125349"
-					(reference "#PWR17")
+					(reference "#PWR60")
 					(unit 1)
 				)
 				(path "/3d1a8eae-9f4e-4ae3-8a80-a6e3408e9f8d/471bb7b7-cd79-4b45-b5fa-ce18ba37980a"
-					(reference "#PWR11")
+					(reference "#PWR52")
 					(unit 1)
 				)
 				(path "/3d1a8eae-9f4e-4ae3-8a80-a6e3408e9f8d/77ed2068-19f4-4838-81a2-88ec2b717aa2"
-					(reference "#PWR20")
+					(reference "#PWR64")
 					(unit 1)
 				)
 				(path "/3d1a8eae-9f4e-4ae3-8a80-a6e3408e9f8d/ed3c01a7-dc5a-420d-9436-94dfdef482d0"
-					(reference "#PWR14")
+					(reference "#PWR56")
 					(unit 1)
 				)
@@
 		(dnp no)
 		(fields_autoplaced yes)
-		(property "Reference" "#PWR10"
+		(property "Reference" "#PWR51"
 			(at 185.42 144.78 0)
 			(effects
@@
 			(project "minimal_ad74413r"
 				(path "/3d1a8eae-9f4e-4ae3-8a80-a6e3408e9f8d/215a75b8-84cc-467b-b211-24faa4125349"
-					(reference "#PWR16")
+					(reference "#PWR59")
 					(unit 1)
 				)
 				(path "/3d1a8eae-9f4e-4ae3-8a80-a6e3408e9f8d/471bb7b7-cd79-4b45-b5fa-ce18ba37980a"
-					(reference "#PWR10")
+					(reference "#PWR51")
 					(unit 1)
 				)
 				(path "/3d1a8eae-9f4e-4ae3-8a80-a6e3408e9f8d/77ed2068-19f4-4838-81a2-88ec2b717aa2"
-					(reference "#PWR19")
+					(reference "#PWR63")
 					(unit 1)
 				)
 				(path "/3d1a8eae-9f4e-4ae3-8a80-a6e3408e9f8d/ed3c01a7-dc5a-420d-9436-94dfdef482d0"
-					(reference "#PWR12")
+					(reference "#PWR55")
 					(unit 1)
 				)
@@
 		(dnp no)
 		(fields_autoplaced yes)
-		(property "Reference" "#PWR023"
+		(property "Reference" "#PWR54"
 			(at 241.3 132.08 0)
 			(effects
@@
 			(project "minimal_ad74413r"
 				(path "/3d1a8eae-9f4e-4ae3-8a80-a6e3408e9f8d/215a75b8-84cc-467b-b211-24faa4125349"
-					(reference "#PWR025")
+					(reference "#PWR62")
 					(unit 1)
 				)
 				(path "/3d1a8eae-9f4e-4ae3-8a80-a6e3408e9f8d/471bb7b7-cd79-4b45-b5fa-ce18ba37980a"
-					(reference "#PWR023")
+					(reference "#PWR54")
 					(unit 1)
 				)
 				(path "/3d1a8eae-9f4e-4ae3-8a80-a6e3408e9f8d/77ed2068-19f4-4838-81a2-88ec2b717aa2"
-					(reference "#PWR026")
+					(reference "#PWR66")
 					(unit 1)
 				)
 				(path "/3d1a8eae-9f4e-4ae3-8a80-a6e3408e9f8d/ed3c01a7-dc5a-420d-9436-94dfdef482d0"
-					(reference "#PWR024")
+					(reference "#PWR58")
 					(unit 1)
 				)
@@
 		(dnp no)
 		(fields_autoplaced yes)
-		(property "Reference" "#PWR13"
+		(property "Reference" "#PWR53"
 			(at 228.6 132.08 0)
 			(effects
@@
 			(project "minimal_ad74413r"
 				(path "/3d1a8eae-9f4e-4ae3-8a80-a6e3408e9f8d/215a75b8-84cc-467b-b211-24faa4125349"
-					(reference "#PWR18")
+					(reference "#PWR61")
 					(unit 1)
 				)
 				(path "/3d1a8eae-9f4e-4ae3-8a80-a6e3408e9f8d/471bb7b7-cd79-4b45-b5fa-ce18ba37980a"
-					(reference "#PWR13")
+					(reference "#PWR53")
 					(unit 1)
 				)
 				(path "/3d1a8eae-9f4e-4ae3-8a80-a6e3408e9f8d/77ed2068-19f4-4838-81a2-88ec2b717aa2"
-					(reference "#PWR21")
+					(reference "#PWR65")
 					(unit 1)
 				)
 				(path "/3d1a8eae-9f4e-4ae3-8a80-a6e3408e9f8d/ed3c01a7-dc5a-420d-9436-94dfdef482d0"
-					(reference "#PWR15")
+					(reference "#PWR57")
 					(unit 1)
 				)
@@
 		(dnp no)
 		(fields_autoplaced yes)
-		(property "Reference" "D12"
+		(property "Reference" "D4"
 			(at 245.11 113.0299 90)
 			(effects
@@
 			(project "minimal_ad74413r"
 				(path "/3d1a8eae-9f4e-4ae3-8a80-a6e3408e9f8d/215a75b8-84cc-467b-b211-24faa4125349"
-					(reference "D14")
+					(reference "D1")
 					(unit 1)
 				)
 				(path "/3d1a8eae-9f4e-4ae3-8a80-a6e3408e9f8d/471bb7b7-cd79-4b45-b5fa-ce18ba37980a"
-					(reference "D12")
+					(reference "D4")
 					(unit 1)
 				)
 				(path "/3d1a8eae-9f4e-4ae3-8a80-a6e3408e9f8d/77ed2068-19f4-4838-81a2-88ec2b717aa2"
-					(reference "D15")
+					(reference "D3")
 					(unit 1)
 				)
 				(path "/3d1a8eae-9f4e-4ae3-8a80-a6e3408e9f8d/ed3c01a7-dc5a-420d-9436-94dfdef482d0"
-					(reference "D13")
-					(unit 1)
-				)
+					(reference "D2")
+					(unit 1)
+				)
